Commit message: Initial commit (Starting from vision_ws)

File: ur_description/urdf/ur5_robot.urdf.xacro (robot description, xacro)
@@ -2,4 +2,5 @@
 <robot xmlns:xacro="http://ros.org/wiki/xacro"
        name="ur5" >
+  <property name="M_PI" value="3.14159265359" />
   <!-- common stuff -->
   <xacro:include filename="$(find ur_description)/urdf/common.gazebo.xacro" />
@@ -12,5 +13,5 @@
     <parent link="world" />
     <child link = "base_link" />
-    <origin xyz="0.0 0.0 0.0" rpy="0.0 0.0 0.0" />
+    <origin xyz="10.0 0.0 0.0" rpy="0.0 0.0 0.0" />
   </joint>
 </robot>
